Commit message: limits geändert

File: urdf/collissionur5.urdf.xacro (robot description, xacro)
@@ -96,5 +96,5 @@
       </xacro:unless>
       <xacro:if value="${joint_limited}">
-        <limit lower="${-pi-pi/2}" upper="${-pi/4}" effort="150.0" velocity="3.15"/>
+        <limit lower="${-pi/2}" upper="${pi}" effort="150.0" velocity="3.15"/>
       </xacro:if>
       <dynamics damping="0.0" friction="0.0"/>
@@ -220,5 +220,5 @@
       </xacro:unless>
       <xacro:if value="${joint_limited}">
-        <limit lower="${-pi}" upper="${pi}" effort="28.0" velocity="3.2"/>
+        <limit lower="${-(2*pi)}" upper="${-(pi/2)}" effort="28.0" velocity="3.2"/>
       </xacro:if>
       <dynamics damping="0.0" friction="0.0"/>

File: urdf/tams_setup.urdf.xacro (robot description, xacro)
@@ -38,5 +38,6 @@
     <!-- virtual wall is set to the adapter elements front surface!!! -->
     <!-- measured height of ur5 flange screws is 0.97 and 1.065 -> z=1.0175 -->
-    <origin xyz="0.0 0.722 1.0175" rpy="1.571 0.0 1.571" />
+    <!-- 0.722 auf 0.822 geändert-->
+    <origin xyz="0.0 0.822 1.0175" rpy="1.571 0.0 1.571" />
   </joint>
 </robot>
