Commit message: ur5 limits

File: urdf/ur5.urdf_Kopie.xacro (robot description, xacro)
@@ -189,5 +189,5 @@
       </xacro:unless>
       <xacro:if value="${joint_limited}">
-        <limit lower="${-pi}" upper="${pi}" effort="28.0" velocity="3.2"/>
+        <limit lower="${pi/2}" upper="${pi+pi/2}" effort="28.0" velocity="3.2"/>
       </xacro:if>
       <dynamics damping="0.0" friction="0.0"/>
