Commit message: hand greift immer

File: urdf/ur5.urdf.xacro (robot description, xacro)
@@ -158,5 +158,5 @@
       </xacro:unless>
       <xacro:if value="${joint_limited}">
-        <limit lower="${0}" upper="${pi}" effort="150.0" velocity="3.15"/>
+        <limit lower="${-pi}" upper="${pi}" effort="150.0" velocity="3.15"/>
       </xacro:if>
       <dynamics damping="0.0" friction="0.0"/>
